File: Keyboard_HVC-007/KiCad/Nintendo_Famicom_Keyboard_HVC-007.kicad_pcb (KiCad board)
At the start: 2 copper layers, 99 parts, among them IC1 4017, IC2 4019, IC3 4069, P1 Famicom Extension Port, P4 READ/EAR, P5 WRITE/MIC, SW1 F8, SW10 @, SW11 ;, SW12 :, SW13 ン, SW14 /, SW15 -, SW16 ^, SW17 F6, SW18 O, SW19 L, SW2 RET, SW20 K, SW21 ,, SW22 ., SW23 P, SW24 0, SW25 F5, SW26 I, SW27 U, SW28 J, SW29 M, SW3 [, SW30 N, SW31 9, SW32 8, SW33 F4, SW34 Y, SW35 G, SW36 H, SW37 B, SW38 V, SW39 7, SW4 ], SW40 6, SW41 F3, SW42 T, SW43 R, SW44 D, SW45 F, SW46 C, SW47 5, SW48 4, SW49 F2, SW5 カナ, SW50 W, SW51 S, SW52 A, SW53 X, SW54 Z, SW55 E, SW56 3, SW57 F1, SW58 ESC, SW59 Q, SW6 RH SHIFT, SW60 CTR, SW61 LH SHIFT, SW62 GRPH, SW63 1, SW64 2, SW65 CLR HOME, SW66 UP, SW67 RIGHT, SW68 LEFT, SW69 DOWN, SW7 ￥, SW70 SPACE, SW71 DEL, SW72 INS, SW8 STOP, SW9 F7

Commit message: PCB design progress
Parts:
- added H1: MountingHole, MountingHole:MountingHole_3.2mm_M3, F.Cu at (391.4, 54.8)
- added H2: MountingHole, MountingHole:MountingHole_3.2mm_M3, F.Cu at (391.4, 204.8)
- added H3: MountingHole, MountingHole:MountingHole_3.2mm_M3, F.Cu at (201.4, 54.8)
- added H4: MountingHole, MountingHole:MountingHole_3.2mm_M3, F.Cu at (201.4, 204.8)
- added H5: MountingHole, MountingHole:MountingHole_3.2mm_M3, F.Cu at (25.4, 204.8)
- added H6: MountingHole, MountingHole:MountingHole_3.2mm_M3, F.Cu at (25.4, 54.8)
- moved R2 13.2 mm to (328.9, 71.2)
- moved C3 13.2 mm to (325.1, 81.3)
- moved D10 13.2 mm to (321.3, 81.3)
- moved P4 13.2 mm to (322.0, 63.2)
- moved P5 13.2 mm to (332.9, 63.3)
- moved P1 11.6 mm to (353.2, 68.1)
Routing:
- net /P2_9: track 482.5 -> 345.4 mm
- net /JOY1_{D1}: track 65.1 -> 0.00 mm
- net /JOY2_{D3}: track 62.2 -> 0.00 mm
- net /OUT1: track 75.6 -> 13.5 mm
- net /OUT2: track 48.6 -> 0.00 mm, vias 1 -> 0
- net /GND: track 90.4 -> 53.5 mm
- net /OUT0: track 27.0 -> 3.13 mm
- net Net-(D10-A): track 56.1 -> 38.3 mm
- net Net-(P5-Pad2): track 21.1 -> 3.81 mm
- net Net-(IC3-Pad11): track 12.0 -> 0.00 mm
- net /JOY2_{D4}: track 10.5 -> 0.00 mm
Other:
- board outline added: 380 x 160 mm

Commit message: Initial PCB layout completed
Parts:
- added KB1: Space Bar, PCM_Mounting_Keyboard_Stabilizer:Stabilizer_Cherry_MX_7.00u, F.Cu at (166.5, 189.0)
- C1: value 10µF -> 100nF; footprint Capacitor_THT:CP_Radial_D5.0mm_P2.50mm -> Capacitor_THT:C_Axial_L3.8mm_D2.6mm_P7.50mm_Horizontal
- C5, C6: value 10nF -> 100nF
- moved RA1 92.1 mm to (349.5, 96.8), turned to 0 degrees
- moved IC2 84.4 mm to (354.6, 80.2), turned to 90 degrees
- moved C6 56.8 mm to (350.7, 76.4)
- moved D9 45.6 mm to (259.4, 75.2)
- moved C2 35.5 mm to (269.6, 57.4)
- moved C5 35.5 mm to (269.6, 53.6)
- moved R4 35.5 mm to (269.5, 65.0)
- moved IC1 35.5 mm to (259.4, 53.6)
- moved R3 35.5 mm to (279.7, 61.2)
- moved D5 31.8 mm to (245.4, 71.4)
- moved D1 31.8 mm to (245.4, 58.7)
- moved D2 31.8 mm to (245.4, 56.1)
- moved D3 31.8 mm to (245.4, 61.2)
- moved D4 31.8 mm to (245.4, 68.8)
- moved D6 31.8 mm to (245.4, 53.6)
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Routing:
- net /V_{CC}: track 12.4 -> 169.4 mm
- net /P3_4: track 341.7 -> 486.9 mm
- net /P3_5: track 375.3 -> 508.8 mm
- net /P3_6: track 288.2 -> 408.4 mm
- net /OUT1: track 13.5 -> 115.8 mm, vias 0 -> 2
- net /OUT0: track 3.13 -> 103.9 mm
- net Net-(IC2-KA): track 0.00 -> 89.7 mm, vias 0 -> 1
- net /P2_9: track 345.4 -> 431.7 mm
- net /OUT2: track 0.00 -> 84.1 mm
- net /JOY1_{D1}: track 0.00 -> 76.9 mm
- net /P3_3: track 399.2 -> 473.4 mm
- net /GND: track 53.5 -> 120.3 mm, vias 0 -> 32
- net /P3_2: track 356.8 -> 412.7 mm, vias 0 -> 1
- net Net-(P5-Pad2): track 3.81 -> 57.5 mm
- net /P3_1: track 321.2 -> 365.1 mm
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- added copper zone on B.Cu, net /GND
- added copper zone on F.Cu, net /GND
Other:
- board text added: "Keyboard HVC-007 for Nintendo Family Computer Brett Hallen, Dec 2025 Rev. A"
- board text added: "ニンテンドーファミリーコンピュータ用 キーボード「HVC-007」"
- board text removed: "WORK IN PROGRESS"

Commit message: Updated value text visibility
Parts:
- SW2: value RET -> RETURN
Routing:
- net /GND: vias 32 -> 20
